Commit message: Typo correction

File: turtlebot3/turtlebot3_description/urdf/turtlebot3_burger_rrt_urdf.xacro (robot description, xacro)
@@ -31,5 +31,5 @@
     </inertial>
   </link>
-  <joint name="robot_1/wheel_left_joint" type="continuous">
+  <joint name="wheel_left_joint" type="continuous">
     <parent link="robot_1/base_link"/>
     <child link="robot_1/wheel_left_link"/>
@@ -59,5 +59,5 @@
       </inertial>
   </link>
-  <joint name="robot_1/wheel_right_joint" type="continuous">
+  <joint name="wheel_right_joint" type="continuous">
     <parent link="robot_1/base_link"/>
     <child link="robot_1/wheel_right_link"/>
